File: IFT-C3.kicad_sch (KiCad schematic)
At the start: 40 parts, among them IC1 DIO5508XS8, J2 Conn_01x10_Pin, J3 USB4085-GF-A_REVB, J4 Conn_01x10_Pin, J5 SJ-3523-SMT-TR, J7 Conn_01x02, U1 AZ1117-3.3, U2 ESP32-C3-WROOM-02

Commit message: WIP v2024
Parts:
- added J1: Conn_01x04_Socket, footprints:SSD1306_module, symbol Connector:Conn_01x04_Socket
- added SW1: SW_Push_Dual, footprints:PTS526SM15SMTR2LFS, symbol Switch:SW_Push_Dual
- added U3: MAX98357A, Package_DFN_QFN:TQFN-16-1EP_3x3mm_P0.5mm_EP1.23x1.23mm, symbol Audio:MAX98357A
- gave numbers to parts that had none: 2
Connections:
- net +3.3V: now also J1.2 (Pin_2)
- net +BATT: now also J7.1 (Pin_1); no longer C1.1, U1.3 (VI)
- net GND: now also J1.1 (Pin_1), SW1.1, SW1.3
- net +BATT_after_switch: now reaches S1.C1 (NO)
- net +BATT_after_switch: now also C1.1, U1.3 (VI); no longer J7.1 (Pin_1)
- net Button/NO: no longer names the net of C3.1, R3.1, U2.2 (EN/CHIP_PU)
- net Button/NO: now also SW1.2, SW1.4
- new net: U3.11 (GND), U3.15 (GND), U3.3 (GND)
- new net: U3.7 (VDD), U3.8 (VDD)
- new net SCL: J1.3 (Pin_3)
- new net SDA: J1.4 (Pin_4)
Other:
- removed sheet Button
- removed sheet Button1
- added sheet Keyboard Matrix (keyboard_matrix.kicad_sch)
- note added: "Connector to screen"
- note added: "Reset"
- moved on the sheet: J7, JP6, R1, S1
