File: pwm_filter.kicad_sch (KiCad schematic)
At the start: 3 parts

Commit message: WIP, routed
Parts:
- renumbered C8 to C10, C9 to C11, R9 to R10
Changed lines of the file:
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@@
 		(dnp no)
 		(fields_autoplaced yes)
-		(property "Reference" "#PWR035"
+		(property "Reference" "#PWR043"
 			(at 148.59 97.79 0)
 			(effects
@@
 		(dnp no)
 		(fields_autoplaced yes)
-		(property "Reference" "C9"
+		(property "Reference" "C11"
 			(at 156.591 74.93 90)
 			(effects
@@
 		(on_board yes)
 		(dnp no)
-		(property "Reference" "R9"
+		(property "Reference" "R10"
 			(at 142.24 82.55 90)
 			(effects
@@
 		(dnp no)
 		(fields_autoplaced yes)
-		(property "Reference" "C8"
+		(property "Reference" "C10"
 			(at 152.4 86.36 0)
 			(effects

Commit message: Uniformed values for R and C for a better BOM
Parts:
- C10: value 100nF -> 100n
Changed lines of the file:
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@@
 			)
 		)
-		(property "Value" "100nF"
+		(property "Value" "100n"
 			(at 152.4 88.9 0)
 			(effects
